File: балансир/балансир.sch (KiCad schematic (older format))
At the start: 48 parts

Commit message: есть схема, но нет решения по связи
Parts:
- added C?: 4.7мкФ, 1210, N_RLC:Конденсатор_SMD_1210, symbol elements:Конденсатор_керамический
- added DD?: 5559ИН10_28(UART-RS485), N_DD:SO-8, symbol elements:5559ИН10_28(UART-RS485)
- added XТ? (x2): Клеммник_х2, N_X:Клеммник_х2_шаг5, symbol elements:Клеммник_х2
Connections:
- net labels added: A, B, EnRS, RX, TX
- wire segments 173 -> 192
Changed lines of the file:
@@
 Wire Wire Line
 	12675 7750 12375 7750
-Text Label 12675 8950 0    50   ~ 0
+Text Label 12825 8950 0    50   ~ 0
 RES
 Wire Wire Line
-	12675 8950 12625 8950
+	12825 8950 12775 8950
 Text Label 10025 9150 2    50   ~ 0
 MOSI
@@
 L elements:Резистор_0,125Вт R?
 U 1 1 5C5985AE
-P 13350 9050
-F 0 "R?" H 13225 8925 60  0000 L CNN
-F 1 "20к, 0805" H 13075 9200 60  0000 L CNN
-F 2 "N_RLC:Резистор_SMD_0805_0,125Вт" H 13350 9050 60  0001 C CNN
-F 3 "" H 13350 9050 60  0001 C CNN
-	1    13350 9050
+P 13500 9050
+F 0 "R?" H 13375 8925 60  0000 L CNN
+F 1 "20к, 0805" H 13225 9200 60  0000 L CNN
+F 2 "N_RLC:Резистор_SMD_0805_0,125Вт" H 13500 9050 60  0001 C CNN
+F 3 "" H 13500 9050 60  0001 C CNN
+	1    13500 9050
 	-1   0    0    1
 $EndComp
-Text Label 14000 9050 0    50   ~ 0
-VCC
-Wire Wire Line
-	14000 9050 13750 9050
-Wire Wire Line
-	12950 9050 12625 9050
-Wire Wire Line
-	12625 9050 12625 8950
-Connection ~ 12625 8950
-Wire Wire Line
-	12625 8950 12375 8950
+Text Label 14150 9050 0    50   ~ 0
+VCC
+Wire Wire Line
+	14150 9050 13900 9050
+Wire Wire Line
+	13100 9050 12775 9050
+Wire Wire Line
+	12775 9050 12775 8950
+Connection ~ 12775 8950
 $Comp
 L elements:Резистор_0,125Вт R?
@@
 Wire Wire Line
 	13650 8250 13650 8450
+$Comp
+L elements:5559ИН10_28(UART-RS485) DD?
+U 1 1 5C51CC22
+P 6000 9400
+F 0 "DD?" H 6200 9925 60  0000 C CNN
+F 1 "5559ИН10_28(UART-RS485)" H 6025 8875 60  0000 C CNN
+F 2 "N_DD:SO-8" H 6000 9400 60  0001 C CNN
+F 3 "" H 6000 9400 60  0001 C CNN
+	1    6000 9400
+	1    0    0    -1
+$EndComp
+Wire Wire Line
+	5250 9400 5000 9400
+Wire Wire Line
+	5000 9400 5000 9250
+Wire Wire Line
+	5000 9250 5250 9250
+Wire Wire Line
+	5000 9250 4800 9250
+Connection ~ 5000 9250
+Wire Wire Line
+	5250 9550 4800 9550
+Wire Wire Line
+	7200 9050 6750 9050
+Text Label 7200 9050 0    50   ~ 0
+RX
+Wire Wire Line
+	12525 9050 12375 9050
+Wire Wire Line
+	12375 8950 12775 8950
+Text Label 4800 9550 2    50   ~ 0
+TX
+Wire Wire Line
+	12525 9150 12375 9150
+Text Label 4800 9250 2    50   ~ 0
+EnRS
+Wire Wire Line
+	12525 9250 12375 9250
+$Comp
+L elements:Конденсатор_керамический C?
+U 1 1 5C56EAA5
+P 7700 9350
+F 0 "C?" V 7650 9400 60  0000 L CNN
+F 1 "4.7мкФ, 1210" V 7825 9400 60  0000 L CNN
+F 2 "N_RLC:Конденсатор_SMD_1210" H 7700 9350 60  0001 C CNN
+F 3 "" H 7700 9350 60  0001 C CNN
+	1    7700 9350
+	0    1    1    0
+$EndComp
+Text Label 7700 9600 0    50   ~ 0
+0В
+Wire Wire Line
+	7700 9450 7700 9600
+Text Label 7700 9150 0    50   ~ 0
+VCC
+Wire Wire Line
+	7700 9150 7700 9300
+Wire Wire Line
+	7200 9600 6750 9600
+Wire Wire Line
+	7200 9750 6750 9750
+Text Label 7200 9750 0    50   ~ 0
+VCC
+Text Label 7200 9600 0    50   ~ 0
+0В
+Wire Wire Line
+	7200 9250 6750 9250
+Text Label 7200 9250 0    50   ~ 0
+A
+Wire Wire Line
+	7200 9400 6750 9400
+Text Label 7200 9400 0    50   ~ 0
+B
+$Comp
+L elements:Клеммник_х2 XТ?
+U 1 1 5C522BAD
+P 8075 10050
+F 0 "XТ?" H 7936 10256 60  0000 C CNN
+F 1 "Клеммник_х2" H 8025 9675 60  0001 C CNN
+F 2 "N_X:Клеммник_х2_шаг5" H 8075 10050 60  0001 C CNN
+F 3 "" H 8075 10050 60  0001 C CNN
+	1    8075 10050
+	1    0    0    -1
+$EndComp
+Wire Wire Line
+	8525 10050 8075 10050
+Text Label 8525 10050 0    50   ~ 0
+A
+Wire Wire Line
+	8525 10250 8075 10250
+Text Label 8525 10250 0    50   ~ 0
+B
+$Comp
+L elements:Клеммник_х2 XТ?
+U 1 1 5C533893
+P 8075 10650
+F 0 "XТ?" H 7936 10856 60  0000 C CNN
+F 1 "Клеммник_х2" H 8025 10275 60  0001 C CNN
+F 2 "N_X:Клеммник_х2_шаг5" H 8075 10650 60  0001 C CNN
+F 3 "" H 8075 10650 60  0001 C CNN
+	1    8075 10650
+	1    0    0    -1
+$EndComp
+Wire Wire Line
+	8525 10650 8075 10650
+Wire Wire Line
+	8525 10850 8075 10850
+Text Label 8525 10650 0    50   ~ 0
+VCC
+Text Label 8525 10850 0    50   ~ 0
+0В
+Text Label 12525 9050 0    50   ~ 0
+RX
+Text Label 12525 9150 0    50   ~ 0
+TX
+Text Label 12525 9250 0    50   ~ 0
+EnRS
 $EndSCHEMATC

Commit message: добавлена STM32
Parts:
- removed XS?: Плюс, symbol elements:отверстие_под_пайку
- removed XS?: Средняя точка, symbol elements:отверстие_под_пайку
- added C11, C12, C? (x4): 4.7мкФ, 1210, N_RLC:Конденсатор_SMD_1210, symbol elements:Конденсатор_керамический
- added DA1, DA2: МОП-реле_КР293КП4, MOTOR_DD:DIP8, symbol elements:МОП-реле_КР293КП4
- added DD?: STM32F030F4P6(TSSOP-20), symbol elements:STM32F030F4P6(TSSOP-20)
- added G?: стабилизатор_нерегулируемый_MC78LC33NTRG, N_G:Преобразователь_LM2703_SOT-23-5, symbol elements:стабилизатор_нерегулируемый_MC78LC33NTRG
- added R11, R12, R14, R15, R16, R17, R6, R9: Резистор_0,125Вт, N_RLC:Резистор_SMD_0805_0,125Вт, symbol elements:Резистор_0,125Вт
- added R?: 20к, 0805, N_RLC:Резистор_SMD_0805_0,125Вт, symbol elements:Резистор_0,125Вт
- added RK1, RK2: Термистор, symbol elements:Термистор
- added X1: Клеммник_х2, N_X:Клеммник_х2_шаг5, symbol elements:Клеммник_х2
- X5: renamed from XS?; value Средняя точка -> Средняя точка(M12); footprint (none) -> N_X:Отверстие_М12
- X6: renamed from XS?; value Минус -> Минус(M12); footprint (none) -> N_X:Отверстие_М12
- XP1: renamed from XP?; footprint (none) -> N_X:Вилка_PLD6_вертикальная
- gave numbers to parts that had none: 47
Connections:
- net labels added: +5, ADC0, ADC1, EnRS_ext, GND, RX_ext, TX_ext
- wire segments 192 -> 277
- no-connect marks 2 -> 6

Commit message: не решен вопрос стабильного питания, не убран старый контроллер
Parts:
- removed C? (x2): 4.7мкФ, 1210, N_RLC:Конденсатор_SMD_1210, symbol elements:Конденсатор_керамический
- removed G1: стабилизатор_нерегулируемый_LM2931, N_G:Стабилизатор_корпус_TO-92, symbol elements:стабилизатор_нерегулируемый_LM2931
- added C? (x2): 4.7мкФ, 1210, N_RLC:Конденсатор_SMD_1210, symbol elements:Конденсатор_керамический
- added R?: 20к, 0805, N_RLC:Резистор_SMD_0805_0,125Вт, symbol elements:Резистор_0,125Вт
Connections:
- net labels added: ADC5_6V, ADCT2, ADC_3V, ADC_T1, BOOT_mode, CLK, DIO, RXboot_SDA, TXboot_SCL
- wire segments 277 -> 281

Commit message: atmega8 заменена на stm32 разводка не готова
Parts:
- removed C14, C15, C16, C17: 4.7мкФ, 1210, N_RLC:Конденсатор_SMD_1210, symbol elements:Конденсатор_керамический
- removed DD1: ATmega8A-AU, N_DD:микросхема_ATMEGA-8-161AU, symbol elements:ATmega8A-AU
- removed R13: 20к, 0805, N_RLC:Резистор_SMD_0805_0,125Вт, symbol elements:Резистор_0,125Вт
- added C18, C19: 12Ф, 0603, N_RLC:Конденсатор_SMD_0603, symbol elements:Конденсатор_керамический
- added HL1: Светодиод, N_VD_HL:Светодиод_SMD_0603, symbol elements:Светодиод
- added K1, K2: 1437566-3 (FSMSM), N_X:Кнопка_FSMSM, symbol elements:кнопка
- added R18: Резистор_0,125Вт, N_RLC:Резистор_SMD_0805_0,125Вт, symbol elements:Резистор_0,125Вт
- added X4: перемычка_разрывная, N_RLC:Конденсатор_SMD_0603, symbol elements:перемычка_разрывная
- added XP2: Вилка_PLS4, N_X:Вилка_PLS4_вертикальная, symbol elements:Вилка_PLS4
- added XP3, XP4: Вилка_PLS10, N_X:Вилка_PLS10_вертикальная, symbol elements:Вилка_PLS10
- C13, C14, C16, C17: renamed from C?; value 4.7мкФ, 1210 -> 4.7мкФ, 0805; footprint N_RLC:Конденсатор_SMD_1210 -> N_RLC:Конденсатор_SMD_0805
- DD2: renamed from DD?; footprint (none) -> N_DD:SSOP-20
- gave numbers to parts that had none: 3
- renumbered C13 to C15, DD2 to DD1, R16 to R19, X5 to X2, X6 to X3, X2 to X5, X3 to X6
Connections:
- net labels added: +5В_эфир, GND_эфир
- net labels removed: +5В, ADC0, ADC1, ADC5, ADC6, GND, MISO, MOSI, SCK
- wire segments 281 -> 282
- no-connect marks 6 -> 4
